File: lednode.sch (EAGLE design)
At the start: 44 parts

Commit message: Finetned lednode schema, laid out components on lednode board, started routing.
Parts:
- removed R4, R5: 10k, rcl:R-EU_R0805
- added LEDS6: (no value), SparkFun-Connectors:M03LONGPADS
- added Q5, Q6: (no value), adafruit:MOSFET-NWAVE
- added RN3: 220R, dp_devices:RESISTOR_ARRAY_4
- added RN4: 10k, dp_devices:RESISTOR_ARRAY_4
- added SPOT5, SPOT6: M025MM, SparkFun-Connectors:M025MM
Connections:
- removed net NEIGHBOR1: NEIGHBOR1.3, U$1.12
- removed net NEIGHBOR2: NEIGHBOR2.3, U$1.A5
- removed net NEIGHBOR3: NEIGHBOR3.3, U$1.A6
- removed net NEIGHBOR4: NEIGHBOR4.3, U$1.A7
- new net DATA_BUS: NEIGHBOR1.3, NEIGHBOR2.3, NEIGHBOR3.3, NEIGHBOR4.3, U$1.A0
- new net LEDSTRIP6: LEDS6.2, U$1.A2
- new net N$1: Q5.D, SPOT5.2
- new net N$11: Q6.D, SPOT6.2
- new net N$12: Q6.G, RN3B.2
- new net N$8: Q5.G, RN3A.2
- new net SENSOR1: RN3C.1, RN4C.2, SENSOR1.2
- new net SENSOR2: RN3D.1, RN4D.2, SENSOR2.2
- new net SPOTLIGHT5: RN3A.1, RN4A.2, U$1.*10
- new net SPOTLIGHT6: RN3B.1, RN4B.2, U$1.*11
- net +12V: now also LEDS6.1, SPOT5.1, SPOT6.1
- net EXTRA_SENSOR1: now also RN3C.2, U$1.A4; no longer R4.2, SENSOR1.2, U$1.A2
- net EXTRA_SENSOR2: now also RN3D.2, U$1.A5; no longer R5.2, SENSOR2.2, U$1.A3
- net GND: now also LEDS6.3, Q5.S, Q6.S, RN4A.1, RN4B.1, RN4C.1, RN4D.1; no longer R4.1, R5.1
- net LEDSTRIP1: now also U$1.4; no longer U$1.2
- net LEDSTRIP2: now also U$1.2; no longer U$1.*3
- net LEDSTRIP3: now also U$1.7; no longer U$1.*5
- net LEDSTRIP5: now also U$1.A1; no longer U$1.7
- net LIGHTLEVEL: now also U$1.A7; no longer U$1.A0
- net PROXIMITY: now also U$1.13; no longer U$1.4
- net SHAKE: now also U$1.12; no longer U$1.13
- net SOUND_ANALOG: now also U$1.A3; no longer U$1.A4
- net SPOTLIGHT1: now also U$1.*3; no longer U$1.*6
- net SPOTLIGHT2: now also U$1.*5; no longer U$1.*9
- net SPOTLIGHT3: now also U$1.*6; no longer U$1.*10
- net SPOTLIGHT4: now also U$1.*9; no longer U$1.*11
- net TEMPERATURE: now also U$1.A6; no longer U$1.A1
Other:
- note removed: "TODO: Add support for 1 or two more led strips?"
- moved on the sheet: H1, H2, H3, H4, LEDS1, LEDS2, LEDS3, LEDS4, LEDS5, NEIGHBOR1, NEIGHBOR2, NEIGHBOR3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

Commit message: Layout and routing done, silkscreens mostly done.
Parts:
- added LOGO3: LOGO-OSHW-8MILX0100-NT, Logo:LOGO-OSHW-8MILX0100-NT
- U$1: device SparkFun-Boards:ARDUINO_PRO_MINI -> SparkFun-Boards-with-arduino-pro-mini-without-connection-pins:ARDUINO_PRO_MINI
Connections:
- removed net SENSOR2: RN3D.1, RN4D.2, SENSOR2.2
- new net N$13: RN1D.1, RN2D.2, SENSOR2.2
- net EXTRA_SENSOR1: now also RN3A.2; no longer RN3C.2
- net EXTRA_SENSOR2: now also RN1D.2; no longer RN3D.2
- net N$10: now also Q5.G, RN3C.2; no longer Q4.G, RN1D.2
- net N$12: now also RN3D.2; no longer RN3B.2
- net N$8: now also Q4.G, RN3B.2; no longer Q5.G, RN3A.2
- net SENSOR1: now also RN3A.1, RN4A.2; no longer RN3C.1, RN4C.2
- net SPOTLIGHT4: now also RN3B.1, RN4B.2; no longer RN1D.1, RN2D.2
- net SPOTLIGHT5: now also RN3C.1, RN4C.2; no longer RN3A.1, RN4A.2
- net SPOTLIGHT6: now also RN3D.1, RN4D.2; no longer RN3B.1, RN4B.2
Other:
- moved on the sheet: H1, H2, H3, H4, RN1D, RN2D, RN3A, RN3B, RN3C, RN3D, RN4A, RN4B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
Changed lines of the file:
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@@
 <part name="SUPPLY2" library="supply2" deviceset="+5V" device=""/>
 <part name="SUPPLY6" library="supply2" deviceset="GND" device=""/>
-<part name="U$1" library="SparkFun-Boards" deviceset="ARDUINO_PRO_MINI" device=""/>
+<part name="U$1" library="SparkFun-Boards-with-arduino-pro-mini-without-connection-pins" deviceset="ARDUINO_PRO_MINI" device=""/>
 <part name="LEDS1" library="SparkFun-Connectors" deviceset="M03" device="LONGPADS"/>
 <part name="LEDS2" library="SparkFun-Connectors" deviceset="M03" device="LONGPADS"/>
@@
 <part name="SUPPLY61" library="supply2" deviceset="+12V" device=""/>
 <part name="SUPPLY63" library="supply2" deviceset="GND" device=""/>
+<part name="LOGO3" library="Logo" deviceset="LOGO-OSHW-8MIL" device="X0100-NT"/>
 </parts>
 <sheets>
@@
 <instance part="C2" gate="G$1" x="-20.32" y="-58.42"/>
 <instance part="PHOTOCELL" gate="G$1" x="-157.48" y="-45.72" rot="R90"/>
-<instance part="H1" gate="G$1" x="-17.78" y="-111.76"/>
-<instance part="H2" gate="G$1" x="10.16" y="-111.76"/>
-<instance part="H3" gate="G$1" x="-17.78" y="-119.38"/>
-<instance part="H4" gate="G$1" x="10.16" y="-119.38"/>
+<instance part="H1" gate="G$1" x="-20.32" y="-106.68"/>
+<instance part="H2" gate="G$1" x="7.62" y="-106.68"/>
+<instance part="H3" gate="G$1" x="-20.32" y="-114.3"/>
+<instance part="H4" gate="G$1" x="7.62" y="-114.3"/>
 <instance part="SUPPLY1" gate="+12V" x="81.28" y="35.56" rot="R90"/>
 <instance part="SUPPLY3" gate="+12V" x="81.28" y="17.78" rot="R90"/>
@@
 <instance part="RN1" gate="B" x="144.78" y="33.02"/>
 <instance part="RN1" gate="C" x="144.78" y="5.08"/>
-<instance part="RN1" gate="D" x="144.78" y="-22.86"/>
+<instance part="RN1" gate="D" x="-68.58" y="-71.12"/>
 <instance part="RN1" gate="A" x="144.78" y="60.96"/>
 <instance part="RN2" gate="B" x="139.7" y="27.94" rot="R90"/>
 <instance part="RN2" gate="C" x="139.7" y="0" rot="R90"/>
-<instance part="RN2" gate="D" x="139.7" y="-27.94" rot="R90"/>
+<instance part="RN2" gate="D" x="-81.28" y="-76.2" rot="R90"/>
 <instance part="RN2" gate="A" x="139.7" y="55.88" rot="R90"/>
 <instance part="SUPPLY19" gate="GND" x="139.7" y="48.26"/>
@@
 <instance part="SUPPLY61" gate="+12V" x="154.94" y="-66.04"/>
 <instance part="SUPPLY63" gate="GND" x="139.7" y="-91.44"/>
-<instance part="RN3" gate="A" x="144.78" y="-50.8"/>
-<instance part="RN3" gate="B" x="144.78" y="-78.74"/>
-<instance part="RN3" gate="C" x="-71.12" y="-38.1"/>
-<instance part="RN4" gate="A" x="139.7" y="-55.88" rot="R90"/>
-<instance part="RN4" gate="B" x="139.7" y="-83.82" rot="R90"/>
-<instance part="RN4" gate="C" x="-81.28" y="-43.18" rot="R90"/>
-<instance part="RN4" gate="D" x="-81.28" y="-76.2" rot="R90"/>
-<instance part="RN3" gate="D" x="-71.12" y="-71.12"/>
+<instance part="RN3" gate="A" x="-68.58" y="-38.1"/>
+<instance part="RN3" gate="B" x="144.78" y="-22.86"/>
+<instance part="RN3" gate="C" x="144.78" y="-50.8"/>
+<instance part="RN4" gate="A" x="-81.28" y="-43.18" rot="R90"/>
+<instance part="RN4" gate="B" x="139.7" y="-27.94" rot="R90"/>
+<instance part="RN4" gate="C" x="139.7" y="-55.88" rot="R90"/>
+<instance part="RN4" gate="D" x="139.7" y="-83.82" rot="R90"/>
+<instance part="RN3" gate="D" x="144.78" y="-78.74"/>
+<instance part="LOGO3" gate="G$1" x="2.54" y="-129.54"/>
 </instances>
 <busses>
@@
 </segment>
 <segment>
-<pinref part="RN2" gate="D" pin="1"/>
-<pinref part="SUPPLY22" gate="GND" pin="GND"/>
-</segment>
-<segment>
 <pinref part="PIR" gate="G$1" pin="1"/>
 <pinref part="SUPPLY30" gate="GND" pin="GND"/>
@@
 </segment>
 <segment>
+<pinref part="SUPPLY63" gate="GND" pin="GND"/>
+<pinref part="RN4" gate="D" pin="1"/>
+</segment>
+<segment>
 <pinref part="SUPPLY60" gate="GND" pin="GND"/>
+<pinref part="RN4" gate="C" pin="1"/>
+</segment>
+<segment>
+<pinref part="SUPPLY22" gate="GND" pin="GND"/>
+<pinref part="RN4" gate="B" pin="1"/>
+</segment>
+<segment>
+<pinref part="SUPPLY37" gate="GND" pin="GND"/>
 <pinref part="RN4" gate="A" pin="1"/>
 </segment>
 <segment>
-<pinref part="SUPPLY63" gate="GND" pin="GND"/>
-<pinref part="RN4" gate="B" pin="1"/>
-</segment>
-<segment>
 <pinref part="SUPPLY49" gate="GND" pin="GND"/>
-<pinref part="RN4" gate="D" pin="1"/>
-</segment>
-<segment>
-<pinref part="SUPPLY37" gate="GND" pin="GND"/>
-<pinref part="RN4" gate="C" pin="1"/>
+<pinref part="RN2" gate="D" pin="1"/>
 </segment>
 </net>
@@
 <net name="SPOTLIGHT4" class="0">
 <segment>
-<wire x1="139.7" y1="-22.86" x2="124.46" y2="-22.86" width="0.1524" layer="91"/>
 <label x="124.46" y="-22.86" size="1.778" layer="95"/>
-<pinref part="RN2" gate="D" pin="2"/>
-<pinref part="RN1" gate="D" pin="1"/>
+<pinref part="RN3" gate="B" pin="1"/>
+<wire x1="124.46" y1="-22.86" x2="139.7" y2="-22.86" width="0.1524" layer="91"/>
+<pinref part="RN4" gate="B" pin="2"/>
 <junction x="139.7" y="-22.86"/>
 </segment>
@@
 <pinref part="Q3" gate="G$1" pin="G"/>
 <pinref part="RN1" gate="C" pin="2"/>
-</segment>
-</net>
-<net name="N$10" class="0">
-<segment>
-<pinref part="Q4" gate="G$1" pin="G"/>
-<pinref part="RN1" gate="D" pin="2"/>
 </segment>
 </net>
@@
 </segment>
 <segment>
-<pinref part="RN3" gate="C" pin="2"/>
-<wire x1="-66.04" y1="-38.1" x2="-43.18" y2="-38.1" width="0.1524" layer="91"/>
+<wire x1="-63.5" y1="-38.1" x2="-43.18" y2="-38.1" width="0.1524" layer="91"/>
 <label x="-63.5" y="-38.1" size="1.778" layer="95"/>
+<pinref part="RN3" gate="A" pin="2"/>
 </segment>
 </net>
@@
 </segment>
 <segment>
-<pinref part="RN3" gate="D" pin="2"/>
-<wire x1="-66.04" y1="-71.12" x2="-43.18" y2="-71.12" width="0.1524" layer="91"/>
+<wire x1="-63.5" y1="-71.12" x2="-43.18" y2="-71.12" width="0.1524" layer="91"/>
 <label x="-63.5" y="-71.12" size="1.778" layer="95"/>
+<pinref part="RN1" gate="D" pin="2"/>
 </segment>
 </net>
@@
 <net name="SPOTLIGHT5" class="0">
 <segment>
-<wire x1="139.7" y1="-50.8" x2="124.46" y2="-50.8" width="0.1524" layer="91"/>
 <label x="124.46" y="-50.8" size="1.778" layer="95"/>
-<pinref part="RN3" gate="A" pin="1"/>
-<pinref part="RN4" gate="A" pin="2"/>
+<pinref part="RN3" gate="C" pin="1"/>
+<wire x1="124.46" y1="-50.8" x2="139.7" y2="-50.8" width="0.1524" layer="91"/>
+<pinref part="RN4" gate="C" pin="2"/>
 <junction x="139.7" y="-50.8"/>
 </segment>
@@
 <net name="SPOTLIGHT6" class="0">
 <segment>
-<wire x1="139.7" y1="-78.74" x2="124.46" y2="-78.74" width="0.1524" layer="91"/>
 <label x="124.46" y="-78.74" size="1.778" layer="95"/>
-<pinref part="RN3" gate="B" pin="1"/>
-<pinref part="RN4" gate="B" pin="2"/>
+<pinref part="RN3" gate="D" pin="1"/>
+<wire x1="124.46" y1="-78.74" x2="139.7" y2="-78.74" width="0.1524" layer="91"/>
+<pinref part="RN4" gate="D" pin="2"/>
 <junction x="139.7" y="-78.74"/>
 </segment>
@@
 </segment>
 </net>
+<net name="SENSOR1" class="0">
+<segment>
+<pinref part="SENSOR1" gate="G$1" pin="2"/>
+<pinref part="RN4" gate="A" pin="2"/>
+<wire x1="-96.52" y1="-38.1" x2="-81.28" y2="-38.1" width="0.1524" layer="91"/>
+<pinref part="RN3" gate="A" pin="1"/>
+<wire x1="-81.28" y1="-38.1" x2="-73.66" y2="-38.1" width="0.1524" layer="91"/>
+<junction x="-81.28" y="-38.1"/>
+</segment>
+</net>
 <net name="N$8" class="0">
 <segment>
+<pinref part="Q4" gate="G$1" pin="G"/>
+<pinref part="RN3" gate="B" pin="2"/>
+</segment>
+</net>
+<net name="N$10" class="0">
+<segment>
 <pinref part="Q5" gate="G$1" pin="G"/>
-<pinref part="RN3" gate="A" pin="2"/>
+<pinref part="RN3" gate="C" pin="2"/>
 </segment>
 </net>
@@
 <segment>
 <pinref part="Q6" gate="G$1" pin="G"/>
-<pinref part="RN3" gate="B" pin="2"/>
-</segment>
-</net>
-<net name="SENSOR2" class="0">
+<pinref part="RN3" gate="D" pin="2"/>
+</segment>
+</net>
+<net name="N$13" class="0">
 <segment>
 <pinref part="SENSOR2" gate="G$1" pin="2"/>
+<pinref part="RN2" gate="D" pin="2"/>
 <wire x1="-96.52" y1="-71.12" x2="-81.28" y2="-71.12" width="0.1524" layer="91"/>
-<pinref part="RN4" gate="D" pin="2"/>
-<wire x1="-81.28" y1="-71.12" x2="-76.2" y2="-71.12" width="0.1524" layer="91"/>
+<pinref part="RN1" gate="D" pin="1"/>
+<wire x1="-81.28" y1="-71.12" x2="-73.66" y2="-71.12" width="0.1524" layer="91"/>
 <junction x="-81.28" y="-71.12"/>
-<pinref part="RN3" gate="D" pin="1"/>
-</segment>
-</net>
-<net name="SENSOR1" class="0">
-<segment>
-<pinref part="SENSOR1" gate="G$1" pin="2"/>
-<wire x1="-96.52" y1="-38.1" x2="-81.28" y2="-38.1" width="0.1524" layer="91"/>
-<pinref part="RN4" gate="C" pin="2"/>
-<wire x1="-81.28" y1="-38.1" x2="-76.2" y2="-38.1" width="0.1524" layer="91"/>
-<junction x="-81.28" y="-38.1"/>
-<pinref part="RN3" gate="C" pin="1"/>
 </segment>
 </net>
@@
 </sheet>
 </sheets>
+<errors>
+</errors>
 </schematic>
 </drawing>

Commit message: Final touches.
Parts:
- removed H1, H2, H3, H4: MOUNT-HOLE3.2, holes:MOUNT-HOLE3.2
- added GND, RESET, RXI, TXO: M01NOSILK-KIT, SparkFun-Connectors:M01NOSILK-KIT
- PHOTOCELL: device SparkFun:PHOTOCELLPTH -> SparkFun-Sensors:PHOTOCELLPTH
- SOUND_SENSOR: device SparkFun-Connectors:M04PTH -> SparkFun-Connectors:M041X04_NO_SILK
- THERM: device discrete:THERMISTOR_R-7,5 -> discrete-fixed-thermistor-silk:THERMISTOR_R-7,5
Connections:
- new net N$14: TXO.1, U$1.TXO
- new net N$15: RXI.1, U$1.RXI
- new net N$16: RESET.1, U$1.RST
- net GND: now also GND.1
Changed lines of the file:
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@@
 <part name="C3" library="rcl" deviceset="C-EU" device="C1206" value="10 uF"/>
 <part name="C2" library="rcl" deviceset="CPOL-EU" device="E3.5-10" value="100 uF"/>
-<part name="PHOTOCELL" library="SparkFun" deviceset="PHOTOCELL" device="PTH" value="10-20k"/>
-<part name="H1" library="holes" deviceset="MOUNT-HOLE" device="3.2" value="MOUNT-HOLE3.2"/>
-<part name="H2" library="holes" deviceset="MOUNT-HOLE" device="3.2" value="MOUNT-HOLE3.2"/>
-<part name="H3" library="holes" deviceset="MOUNT-HOLE" device="3.2" value="MOUNT-HOLE3.2"/>
-<part name="H4" library="holes" deviceset="MOUNT-HOLE" device="3.2" value="MOUNT-HOLE3.2"/>
+<part name="PHOTOCELL" library="SparkFun-Sensors" deviceset="PHOTOCELL" device="PTH" value="10-20k"/>
 <part name="SUPPLY1" library="supply2" deviceset="+12V" device=""/>
 <part name="SUPPLY3" library="supply2" deviceset="+12V" device=""/>
@@
 <part name="SUPPLY27" library="supply2" deviceset="+5V" device=""/>
 <part name="SUPPLY30" library="supply2" deviceset="GND" device=""/>
-<part name="THERM" library="discrete" deviceset="THERMISTOR_" device="R-7,5" value="10k"/>
+<part name="THERM" library="discrete-fixed-thermistor-silk" deviceset="THERMISTOR_" device="R-7,5" value="10k"/>
 <part name="SUPPLY28" library="supply2" deviceset="+5V" device=""/>
 <part name="SUPPLY29" library="supply2" deviceset="+5V" device=""/>
@@
 <part name="SUPPLY49" library="supply2" deviceset="GND" device=""/>
 <part name="SUPPLY50" library="supply2" deviceset="GND" device=""/>
-<part name="SOUND_SENSOR" library="SparkFun-Connectors" deviceset="M04" device="PTH"/>
+<part name="SOUND_SENSOR" library="SparkFun-Connectors" deviceset="M04" device="1X04_NO_SILK"/>
 <part name="SUPPLY54" library="supply2" deviceset="GND" device=""/>
 <part name="SUPPLY55" library="supply2" deviceset="+5V" device=""/>
@@
 <part name="SUPPLY63" library="supply2" deviceset="GND" device=""/>
 <part name="LOGO3" library="Logo" deviceset="LOGO-OSHW-8MIL" device="X0100-NT"/>
+<part name="TXO" library="SparkFun-Connectors" deviceset="M01" device="NOSILK-KIT" value=""/>
+<part name="RXI" library="SparkFun-Connectors" deviceset="M01" device="NOSILK-KIT" value=""/>
+<part name="RESET" library="SparkFun-Connectors" deviceset="M01" device="NOSILK-KIT" value=""/>
+<part name="GND" library="SparkFun-Connectors" deviceset="M01" device="NOSILK-KIT" value=""/>
+<part name="SUPPLY62" library="supply2" deviceset="GND" device=""/>
 </parts>
 <sheets>
@@
 <instance part="C2" gate="G$1" x="-20.32" y="-58.42"/>
 <instance part="PHOTOCELL" gate="G$1" x="-157.48" y="-45.72" rot="R90"/>
-<instance part="H1" gate="G$1" x="-20.32" y="-106.68"/>
-<instance part="H2" gate="G$1" x="7.62" y="-106.68"/>
-<instance part="H3" gate="G$1" x="-20.32" y="-114.3"/>
-<instance part="H4" gate="G$1" x="7.62" y="-114.3"/>
 <instance part="SUPPLY1" gate="+12V" x="81.28" y="35.56" rot="R90"/>
 <instance part="SUPPLY3" gate="+12V" x="81.28" y="17.78" rot="R90"/>
@@
 <instance part="RN3" gate="D" x="144.78" y="-78.74"/>
 <instance part="LOGO3" gate="G$1" x="2.54" y="-129.54"/>
+<instance part="TXO" gate="G$1" x="-22.86" y="22.86" rot="R270"/>
+<instance part="RXI" gate="G$1" x="-33.02" y="20.32" rot="R270"/>
+<instance part="RESET" gate="G$1" x="-43.18" y="17.78" rot="R270"/>
+<instance part="GND" gate="G$1" x="-53.34" y="15.24" rot="R270"/>
+<instance part="SUPPLY62" gate="GND" x="-53.34" y="5.08"/>
 </instances>
 <busses>
@@
 <pinref part="RN2" gate="D" pin="1"/>
 </segment>
+<segment>
+<pinref part="GND" gate="G$1" pin="1"/>
+<pinref part="SUPPLY62" gate="GND" pin="GND"/>
+</segment>
 </net>
 <net name="+5V" class="0">
@@
 </segment>
 </net>
+<net name="N$14" class="0">
+<segment>
+<pinref part="U$1" gate="G$1" pin="TXO"/>
+<wire x1="-22.86" y1="15.24" x2="-10.16" y2="15.24" width="0.1524" layer="91"/>
+<pinref part="TXO" gate="G$1" pin="1"/>
+</segment>
+</net>
+<net name="N$15" class="0">
+<segment>
+<pinref part="U$1" gate="G$1" pin="RXI"/>
+<wire x1="-33.02" y1="12.7" x2="-10.16" y2="12.7" width="0.1524" layer="91"/>
+<pinref part="RXI" gate="G$1" pin="1"/>
+</segment>
+</net>
+<net name="N$16" class="0">
+<segment>
+<pinref part="U$1" gate="G$1" pin="RST"/>
+<pinref part="RESET" gate="G$1" pin="1"/>
+<wire x1="-10.16" y1="10.16" x2="-43.18" y2="10.16" width="0.1524" layer="91"/>
+</segment>
+</net>

Commit message: Final cleanup and gerber generation.
Parts:
- GND, RESET, RXI, TXO: value M01NOSILK-KIT -> M01SMDNS; device SparkFun-Connectors:M01NOSILK-KIT -> SparkFun-Connectors:M01SMDNS
- Q1, Q2, Q3, Q4, Q5, Q6: value (none) -> AO3402
Other:
- note added: "Breakouts for unused pins"
- moved on the sheet: GND, RESET, RXI, TXO
Changed lines of the file:
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@@
 <part name="C8" library="rcl" deviceset="C-EU" device="C0805" value="100 nF"/>
 <part name="SUPPLY10" library="supply2" deviceset="+12V" device=""/>
-<part name="Q3" library="adafruit" deviceset="MOSFET-N" device="WAVE"/>
-<part name="Q4" library="adafruit" deviceset="MOSFET-N" device="WAVE"/>
-<part name="Q1" library="adafruit" deviceset="MOSFET-N" device="WAVE"/>
-<part name="Q2" library="adafruit" deviceset="MOSFET-N" device="WAVE"/>
+<part name="Q3" library="adafruit" deviceset="MOSFET-N" device="WAVE" value="AO3402"/>
+<part name="Q4" library="adafruit" deviceset="MOSFET-N" device="WAVE" value="AO3402"/>
+<part name="Q1" library="adafruit" deviceset="MOSFET-N" device="WAVE" value="AO3402"/>
+<part name="Q2" library="adafruit" deviceset="MOSFET-N" device="WAVE" value="AO3402"/>
 <part name="SUPPLY11" library="supply2" deviceset="GND" device=""/>
 <part name="SUPPLY12" library="supply2" deviceset="GND" device=""/>
@@
 <part name="SUPPLY56" library="supply2" deviceset="+12V" device=""/>
 <part name="SPOT5" library="SparkFun-Connectors" deviceset="M02" device="5MM"/>
-<part name="Q5" library="adafruit" deviceset="MOSFET-N" device="WAVE"/>
+<part name="Q5" library="adafruit" deviceset="MOSFET-N" device="WAVE" value="AO3402"/>
 <part name="SUPPLY57" library="supply2" deviceset="GND" device=""/>
 <part name="SUPPLY58" library="supply2" deviceset="+12V" device=""/>
@@
 <part name="SUPPLY60" library="supply2" deviceset="GND" device=""/>
 <part name="SPOT6" library="SparkFun-Connectors" deviceset="M02" device="5MM"/>
-<part name="Q6" library="adafruit" deviceset="MOSFET-N" device="WAVE"/>
+<part name="Q6" library="adafruit" deviceset="MOSFET-N" device="WAVE" value="AO3402"/>
 <part name="SUPPLY59" library="supply2" deviceset="GND" device=""/>
 <part name="SUPPLY61" library="supply2" deviceset="+12V" device=""/>
 <part name="SUPPLY63" library="supply2" deviceset="GND" device=""/>
 <part name="LOGO3" library="Logo" deviceset="LOGO-OSHW-8MIL" device="X0100-NT"/>
-<part name="TXO" library="SparkFun-Connectors" deviceset="M01" device="NOSILK-KIT" value=""/>
-<part name="RXI" library="SparkFun-Connectors" deviceset="M01" device="NOSILK-KIT" value=""/>
-<part name="RESET" library="SparkFun-Connectors" deviceset="M01" device="NOSILK-KIT" value=""/>
-<part name="GND" library="SparkFun-Connectors" deviceset="M01" device="NOSILK-KIT" value=""/>
+<part name="TXO" library="SparkFun-Connectors" deviceset="M01" device="SMDNS" value="M01SMDNS"/>
+<part name="RXI" library="SparkFun-Connectors" deviceset="M01" device="SMDNS" value="M01SMDNS"/>
+<part name="RESET" library="SparkFun-Connectors" deviceset="M01" device="SMDNS" value="M01SMDNS"/>
+<part name="GND" library="SparkFun-Connectors" deviceset="M01" device="SMDNS" value="M01SMDNS"/>
 <part name="SUPPLY62" library="supply2" deviceset="GND" device=""/>
 </parts>
@@
 <text x="132.08" y="83.82" size="2.54" layer="91">Spotlight Drivers</text>
 <text x="-111.76" y="15.24" size="2.54" layer="91">Sound Sensor</text>
+<text x="-63.5" y="30.48" size="2.1844" layer="91">Breakouts for unused pins</text>
 </plain>
 <instances>
@@
 <instance part="RN3" gate="D" x="144.78" y="-78.74"/>
 <instance part="LOGO3" gate="G$1" x="2.54" y="-129.54"/>
-<instance part="TXO" gate="G$1" x="-22.86" y="22.86" rot="R270"/>
-<instance part="RXI" gate="G$1" x="-33.02" y="20.32" rot="R270"/>
-<instance part="RESET" gate="G$1" x="-43.18" y="17.78" rot="R270"/>
-<instance part="GND" gate="G$1" x="-53.34" y="15.24" rot="R270"/>
-<instance part="SUPPLY62" gate="GND" x="-53.34" y="5.08"/>
+<instance part="TXO" gate="G$1" x="-30.48" y="25.4" rot="R270"/>
+<instance part="RXI" gate="G$1" x="-40.64" y="25.4" rot="R270"/>
+<instance part="RESET" gate="G$1" x="-50.8" y="25.4" rot="R270"/>
+<instance part="GND" gate="G$1" x="-60.96" y="25.4" rot="R270"/>
+<instance part="SUPPLY62" gate="GND" x="-60.96" y="15.24"/>
 </instances>
 <busses>
@@
 <segment>
 <pinref part="U$1" gate="G$1" pin="TXO"/>
-<wire x1="-22.86" y1="15.24" x2="-10.16" y2="15.24" width="0.1524" layer="91"/>
+<wire x1="-30.48" y1="17.78" x2="-30.48" y2="15.24" width="0.1524" layer="91"/>
+<wire x1="-30.48" y1="15.24" x2="-10.16" y2="15.24" width="0.1524" layer="91"/>
 <pinref part="TXO" gate="G$1" pin="1"/>
 </segment>
@@
 <segment>
 <pinref part="U$1" gate="G$1" pin="RXI"/>
-<wire x1="-33.02" y1="12.7" x2="-10.16" y2="12.7" width="0.1524" layer="91"/>
+<wire x1="-40.64" y1="17.78" x2="-40.64" y2="12.7" width="0.1524" layer="91"/>
+<wire x1="-40.64" y1="12.7" x2="-10.16" y2="12.7" width="0.1524" layer="91"/>
 <pinref part="RXI" gate="G$1" pin="1"/>
 </segment>
@@
 <pinref part="U$1" gate="G$1" pin="RST"/>
 <pinref part="RESET" gate="G$1" pin="1"/>
-<wire x1="-10.16" y1="10.16" x2="-43.18" y2="10.16" width="0.1524" layer="91"/>
-</segment>
-</net>
+<wire x1="-10.16" y1="10.16" x2="-50.8" y2="10.16" width="0.1524" layer="91"/>
+<wire x1="-50.8" y1="10.16" x2="-50.8" y2="17.78" width="0.1524" layer="91"/>
+</segment>
+</net>
