File: controlnode.sch (EAGLE design)
At the start: 29 parts, among them J1 ATX24RH, X1 5566-4, X2 5566-6

Commit message: Started working on powernode. Separated controlnode into an own module.
Parts:
- removed JP10, JP7, JP8, JP9: (no value), SparkFun-Connectors:M03LONGPADS
- removed JP5, JP6: (no value), SparkFun-Connectors:M03-SCREW-5MM
- removed PIR: (no value), SparkFun-Connectors:M03PTH
- added L1, L10, L2, L3, L4, L5, L6, L7, L8, L9: WS2812B, adafruit:WS2812B
- added SW1, SW2: EC12E_SW, switch-alps:EC12E_SW
- added U1: LCD-16X2NOHOLES, SparkFun:LCD-16X2NOHOLES
Connections:
- removed net +5V/2: J1.5V_STDBY, PIR.3, U$1.VCC
- removed net PROXIMITY: PIR.2
- new net 5V_STANDBY: J1.5V_STDBY
- new net N$1: L1.DOUT, L2.DIN
- new net N$10: L1.DIN, U$1.12
- new net N$2: L2.DOUT, L3.DIN
- new net N$20: U$1.*3, U1.A
- new net N$3: L3.DOUT, L4.DIN
- new net N$4: L4.DOUT, L5.DIN
- new net N$5: L5.DOUT, L6.DIN
- new net N$6: L6.DOUT, L7.DIN
- new net N$7: L7.DOUT, L8.DIN
- new net N$8: L8.DOUT, L9.DIN
- new net N$9: L10.DIN, L9.DOUT
- net +5V: now also L1.VDD, L10.VDD, L2.VDD, L3.VDD, L4.VDD, L5.VDD, L6.VDD, L7.VDD, L8.VDD, L9.VDD, U$1.VCC
- net GND: now also L1.GND, L10.GND, L2.GND, L3.GND, L4.GND, L5.GND, L6.GND, L7.GND, L8.GND, L9.GND, U1.K; no longer PIR.1, U$1.GND@2
Other:
- note added: "ColorBar"
- note added: "Inputs"
- note added: "LCD"
- note added: "LCD Contrast Adjustment"
- note added: "Programming Connector"
- note added: "Remote Control Receiver"
- note added: "Speaker?"
- note added: "Switch Potentiometer"
- note added: "Temperature Sensor"
- note added: "Vibration Sensor?"
- note removed: "IR Remote Control Receiver"
- note removed: "Led Node Connectors"
- note removed: "Light level potentiometer"
- note removed: "Main Switch"
- note removed: "PIR Sensor"
- note removed: "Power Led"
- note removed: "Status Leds"
