File: powernode.sch (EAGLE design)
At the start: 29 parts, among them J1 ATX24RH, X1 5566-4, X2 5566-6

Commit message: working on powernode.
Parts:
- removed J1: ATX24RH, SparkFun-Connectors:ATX24RH
- added X3: 5566-24, con-molex:5566-24
Connections:
- net +12V: now also X3-10.S, X3-11.S; no longer J1.12V@0, J1.12V@1
- net +3V3: now also X3-1.S, X3-12.S, X3-13.S, X3-2.S; no longer J1.3.3V@0, J1.3.3V@1, J1.3.3V@2, J1.3.3V@3
- net +5V: now also X3-21.S, X3-22.S, X3-23.S, X3-4.S, X3-6.S; no longer J1.5V@0, J1.5V@1, J1.5V@2, J1.5V@3, J1.5V@4
- net +5V/2: now also X3-9.S; no longer J1.5V_STDBY
- net -12V: now also X3-14.S; no longer J1.-12V
- net GND: now also X3-15.S, X3-17.S, X3-18.S, X3-19.S, X3-24.S, X3-3.S, X3-5.S, X3-7.S; no longer J1.GND@0, J1.GND@1, J1.GND@2, J1.GND@3, J1.GND@4, J1.GND@5, J1.GND@6, J1.GND@7
- net PS_ON: now also X3-16.S; no longer J1.PS_ON
- net PWR_OK: now also X3-8.S; no longer J1.PWR_OK
Other:
- moved on the sheet: S1

Commit message: Working on powernone.
Parts:
- removed C3: 100 nF, rcl:C-EUC0805
- removed JP10, JP7, JP8, JP9: (no value), SparkFun-Connectors:M03LONGPADS
- removed JP5, JP6: (no value), SparkFun-Connectors:M03-SCREW-5MM
- removed S1: (no value), SparkFun:SWITCH-SPSTPTH
- added BLUETOOTH: (no value), SparkFun-Connectors:M06NO_SILK
- added ETHERNET: (no value), con-lsta:FE06-2
- added LED1: (no value), led:LED3MM
- added LEDS1, LEDS2, LEDS3, LEDS4: (no value), SparkFun-Connectors:M03LONGPADS
- added R1: (no value), rcl:R-EU_R0805
- added RN1: 10k, resistor-dil:4R-N0603-ARC
- added SWITCH: (no value), SparkFun-Connectors:M03PTH
- C1: value 100 nF -> 10 uF; device rcl:C-EUC0805 -> rcl:C-EUC1206
- U$1: device SparkFun-Boards:ARDUINO_PRO_MINI -> SparkFun-Boards-with-arduino-pro-mini-without-connection-pins:ARDUINO_PRO_MINI
Connections:
- new net BLUETOOTH_KEY: BLUETOOTH.6
- new net BLUETOOTH_RXD: RN1A.2, U$1.TXO
- new net BLUETOOTH_STATE: BLUETOOTH.1
- new net BLUETOOTH_TXD: BLUETOOTH.3, U$1.RXI
- new net DATA_BUS: JP1.3, JP2.3, JP3.3, JP4.3, U$1.A0
- new net ETHERNET_3_3V: ETHERNET.1
- new net ETHERNET_CLK: ETHERNET.10
- new net ETHERNET_CS: ETHERNET.4, U$1.8
- new net ETHERNET_INT: ETHERNET.9
- new net ETHERNET_SCK: ETHERNET.5, U$1.13
- new net ETHERNET_SI: ETHERNET.6, U$1.*11
- new net ETHERNET_SO: ETHERNET.7, U$1.12
- new net ETHERNET_WAKE_ON_LAN: ETHERNET.8
- new net LEDSTRIP1: LEDS1.2
- new net LEDSTRIP2: LEDS2.2
- new net LEDSTRIP3: LEDS3.2
- new net LEDSTRIP4: LEDS4.2
- new net N$1: U$1.A6
- new net N$10: U$1.A3
- new net N$11: U$1.2
- new net N$12: U$1.*3
- new net N$13: U$1.4
- new net N$14: U$1.*5
- new net N$15: U$1.*6
- new net N$16: U$1.7
- new net N$18: U$1.*9
- new net N$19: U$1.A4
- new net N$2: U$1.A7
- new net N$20: U$1.A5
- new net N$21: BLUETOOTH.2, RN1A.1, RN1B.1
- new net N$22: U$1.RAW
- new net N$3: U$1.*10
- new net N$4: RN1B.2, RN1C.2
- new net N$5: RN1D.1, SWITCH.2
- new net N$6: LED1.A, R1.1
- new net N$8: U$1.A1
- new net N$9: U$1.A2
- new net POWER_SWITCH: RN1D.2
- new net RESET: ETHERNET.3, U$1.RST
- net +12V: now also C4.1, C5.1, C6.1, C7.1, C8.+, C9.+, JP1.1, JP2.1, JP3.1, JP4.1, LEDS1.1, LEDS2.1, LEDS3.1, LEDS4.1, R1.2
- net +5V: no longer C1.1, C2.1, C3.1, C4.1, C5.1, C6.1, C7.1, C8.+, C9.+
- net +5V/2: now also BLUETOOTH.5, C1.1, C2.1, ETHERNET.11, SWITCH.3
- net GND: now also BLUETOOTH.4, ETHERNET.12, ETHERNET.2, JP1.2, JP2.2, JP3.2, JP4.2, LED1.C, LEDS1.3, LEDS2.3, LEDS3.3, LEDS4.3, RN1C.1, SWITCH.1; no longer C3.2, S1.S
- net PS_ON: no longer S1.P
Other:
- note added: "Bluetooth"
- note added: "Ethernet"
- note added: "LED Strip Connectors"
- note added: "Mode selection switch, LCD screen?"
- note removed: "Bluetooth Receiver?"
- note removed: "IR Remote Control Receiver"
- note removed: "LED Strip Connectors (JST 3-Pin, 2.5mm grid, angled)"
- note removed: "Light level potentiometer"
- note removed: "Power Switch"
- note removed: "USB connector to computer (-> use arduino Nano instead of arduino pro mini)"
- moved on the sheet: C1, C2, C4, C5, C6, C7, C8, C9, PIR

Commit message: Working on power / control node.
Parts:
- removed H4: MOUNT-HOLE3.2, holes:MOUNT-HOLE3.2
- added RF_RECEIVER: (no value), SparkFun-Connectors:M041X04_NO_SILK
- added RF_TRANSMITTER: (no value), SparkFun-Connectors:M031X03_NO_SILK
- added SG1: BUZZERPTH-KIT, SparkFun-Electromechanical:BUZZERPTH-KIT
- added SW1: ROTARTY_ENCODER, SparkFun-Electromechanical:ROTARTY_ENCODER
- added U1: LCD-16X2NOHOLES, SparkFun:LCD-16X2NOHOLES
- PIR, SWITCH: device SparkFun-Connectors:M03PTH -> SparkFun-Connectors:M031X03_NO_SILK
Connections:
- new net RF_DATA_IN: RF_RECEIVER.2, RF_RECEIVER.3
- new net RF_DATA_OUT: RF_TRANSMITTER.1
- net +5V/2: now also RF_RECEIVER.1, RF_TRANSMITTER.2
- net GND: now also RF_RECEIVER.4, RF_TRANSMITTER.3
Other:
- note added: "Mode selection switch, LCD screen"
- note removed: "Mode selection switch, LCD screen?"
Changed lines of the file:
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@@
 <part name="H2" library="holes" deviceset="MOUNT-HOLE" device="3.2" value="MOUNT-HOLE3.2"/>
 <part name="H3" library="holes" deviceset="MOUNT-HOLE" device="3.2" value="MOUNT-HOLE3.2"/>
-<part name="H4" library="holes" deviceset="MOUNT-HOLE" device="3.2" value="MOUNT-HOLE3.2"/>
 <part name="X1" library="con-molex" deviceset="5566-4" device=""/>
 <part name="SUPPLY4" library="supply2" deviceset="+12V" device=""/>
@@
 <part name="SUPPLY11" library="supply2" deviceset="+5V/2" device="" value="+5V Standby"/>
 <part name="SUPPLY13" library="supply2" deviceset="GND" device=""/>
-<part name="PIR" library="SparkFun-Connectors" deviceset="M03" device="PTH"/>
+<part name="PIR" library="SparkFun-Connectors" deviceset="M03" device="1X03_NO_SILK"/>
 <part name="SUPPLY14" library="supply2" deviceset="GND" device=""/>
 <part name="X3" library="con-molex" deviceset="5566-24" device=""/>
@@
 <part name="SUPPLY23" library="supply2" deviceset="GND" device=""/>
 <part name="SUPPLY25" library="supply2" deviceset="GND" device=""/>
-<part name="SWITCH" library="SparkFun-Connectors" deviceset="M03" device="PTH"/>
+<part name="SWITCH" library="SparkFun-Connectors" deviceset="M03" device="1X03_NO_SILK"/>
 <part name="SUPPLY24" library="supply2" deviceset="GND" device=""/>
 <part name="SUPPLY26" library="supply2" deviceset="+5V/2" device="" value="+5V Standby"/>
@@
 <part name="SUPPLY43" library="supply2" deviceset="GND" device=""/>
 <part name="SUPPLY44" library="supply2" deviceset="GND" device=""/>
+<part name="RF_RECEIVER" library="SparkFun-Connectors" deviceset="M04" device="1X04_NO_SILK"/>
+<part name="RF_TRANSMITTER" library="SparkFun-Connectors" deviceset="M03" device="1X03_NO_SILK"/>
+<part name="SUPPLY45" library="supply2" deviceset="+5V/2" device="" value="+5V Standby"/>
+<part name="SUPPLY46" library="supply2" deviceset="+5V/2" device="" value="+5V Standby"/>
+<part name="SUPPLY47" library="supply2" deviceset="GND" device=""/>
+<part name="SUPPLY48" library="supply2" deviceset="GND" device=""/>
+<part name="U1" library="SparkFun" deviceset="LCD-16X2" device="NOHOLES" value="LCD-16X2NOHOLES"/>
+<part name="SW1" library="SparkFun-Electromechanical" deviceset="ROTARTY_ENCODER" device=""/>
+<part name="SG1" library="SparkFun-Electromechanical" deviceset="BUZZER" device="PTH-KIT"/>
 </parts>
 <sheets>
@@
 <text x="-58.42" y="-5.08" size="2.54" layer="91">RX / TX radio</text>
 <text x="-93.98" y="127" size="2.54" layer="91">Bluetooth</text>
-<text x="-96.52" y="-7.62" size="2.54" layer="91">Buzzer</text>
+<text x="-99.06" y="0" size="2.54" layer="91">Buzzer</text>
 <text x="106.68" y="2.54" size="2.54" layer="91">Power Led</text>
-<text x="-109.22" y="-17.78" size="2.54" layer="91">Status Leds</text>
+<text x="-205.74" y="22.86" size="2.54" layer="91">Status Leds</text>
 <text x="-142.24" y="104.14" size="2.54" layer="91">Main Switch</text>
 <text x="-157.48" y="43.18" size="2.54" layer="91">PIR Sensor</text>
 <text x="320.04" y="127" size="2.54" layer="91">Led Node Connectors</text>
-<text x="-121.92" y="-33.02" size="2.54" layer="91">Mode selection switch, LCD screen?</text>
+<text x="-170.18" y="0" size="2.54" layer="91">Mode selection switch, LCD screen</text>
 <text x="-63.5" y="45.72" size="2.54" layer="91">Ethernet</text>
 </plain>
@@
 <instance part="H2" gate="G$1" x="180.34" y="55.88"/>
 <instance part="H3" gate="G$1" x="180.34" y="48.26"/>
-<instance part="H4" gate="G$1" x="180.34" y="38.1"/>
 <instance part="X1" gate="-1" x="243.84" y="139.7"/>
 <instance part="X1" gate="-2" x="243.84" y="137.16"/>
@@
 <instance part="SUPPLY43" gate="GND" x="342.9" y="96.52" rot="R270"/>
 <instance part="SUPPLY44" gate="GND" x="342.9" y="116.84" rot="R270"/>
+<instance part="RF_RECEIVER" gate="G$1" x="-45.72" y="-33.02"/>
+<instance part="RF_TRANSMITTER" gate="G$1" x="-48.26" y="-63.5"/>
+<instance part="SUPPLY45" gate="G$1" x="-38.1" y="-35.56" rot="R270"/>
+<instance part="SUPPLY46" gate="G$1" x="-38.1" y="-63.5" rot="R270"/>
+<instance part="SUPPLY47" gate="GND" x="-38.1" y="-60.96" rot="R90"/>
+<instance part="SUPPLY48" gate="GND" x="-38.1" y="-27.94" rot="R90"/>
+<instance part="U1" gate="G$1" x="-121.92" y="-30.48"/>
+<instance part="SW1" gate="G$1" x="-165.1" y="-43.18"/>
+<instance part="SG1" gate="G$1" x="-93.98" y="-10.16"/>
 </instances>
 <busses>
@@
 <pinref part="SUPPLY44" gate="GND" pin="GND"/>
 </segment>
+<segment>
+<pinref part="RF_TRANSMITTER" gate="G$1" pin="3"/>
+<pinref part="SUPPLY47" gate="GND" pin="GND"/>
+</segment>
+<segment>
+<pinref part="RF_RECEIVER" gate="G$1" pin="4"/>
+<pinref part="SUPPLY48" gate="GND" pin="GND"/>
+</segment>
 </net>
 <net name="+5V" class="0">
@@
 <wire x1="-124.46" y1="93.98" x2="-134.62" y2="93.98" width="0.1524" layer="91"/>
 </segment>
+<segment>
+<pinref part="RF_RECEIVER" gate="G$1" pin="1"/>
+<pinref part="SUPPLY45" gate="G$1" pin="+5V/2"/>
+</segment>
+<segment>
+<pinref part="RF_TRANSMITTER" gate="G$1" pin="2"/>
+<pinref part="SUPPLY46" gate="G$1" pin="+5V/2"/>
+</segment>
 </net>
 <net name="PROXIMITY" class="0">
@@
 </segment>
 </net>
+<net name="RF_DATA_OUT" class="0">
+<segment>
+<pinref part="RF_TRANSMITTER" gate="G$1" pin="1"/>
+<wire x1="-40.64" y1="-66.04" x2="-12.7" y2="-66.04" width="0.1524" layer="91"/>
+<label x="-30.48" y="-66.04" size="1.778" layer="95"/>
+</segment>
+</net>
+<net name="RF_DATA_IN" class="0">
+<segment>
+<pinref part="RF_RECEIVER" gate="G$1" pin="3"/>
+<pinref part="RF_RECEIVER" gate="G$1" pin="2"/>
+<wire x1="-40.64" y1="-30.48" x2="-40.64" y2="-33.02" width="0.1524" layer="91"/>
+<wire x1="-40.64" y1="-30.48" x2="-12.7" y2="-30.48" width="0.1524" layer="91"/>
+<junction x="-40.64" y="-30.48"/>
+<label x="-30.48" y="-30.48" size="1.778" layer="95"/>
+</segment>
+</net>

Commit message: Work on powernode.
Parts:
- removed H1, H2, H3: MOUNT-HOLE3.2, holes:MOUNT-HOLE3.2
- removed LED1: (no value), led:LED3MM
- removed LEDS3, LEDS4: (no value), SparkFun-Connectors:M03LONGPADS
- removed SWITCH: (no value), SparkFun-Connectors:M031X03_NO_SILK
- added C10: 100 uF, rcl:CPOL-EUE3.5-10
- added C11, C3: 100 nF, rcl:C-EUC0805
- added CLOCK,TEMP,I2C: (no value), SparkFun:M05PTH
- added IC1: 74HC595D, 74xx-eu:74HC595D
- added POWER_SWITCH: KNC1-101-2P, knc1-101-switch:KNC1-101-2P
- added R2, R4: (no value), rcl:R-EU_R0805
- added R3: 10k, resistor:R-TRIMM3296W
- added R5: (4k), rcl:R-EU_R0805
- added STATUS_LED: (no value), led:DUOLED-RG-C
- R1: value (none) -> (4k)
- X1: device con-molex:5566-4 -> con-molex--with-atx-connectors-without-side-screws:5566-4
- X2: device con-molex:5566-6 -> con-molex--with-atx-connectors-without-side-screws:5566-6
- X3: device con-molex:5566-24 -> con-molex--with-atx-connectors-without-side-screws:5566-24
Connections:
- removed net LEDSTRIP3: LEDS3.2
- removed net LEDSTRIP4: LEDS4.2
- removed net N$12: U$1.*3
- removed net N$13: U$1.4
- removed net N$14: U$1.*5
- removed net N$15: U$1.*6
- removed net N$16: U$1.7
- removed net N$18: U$1.*9
- removed net N$19: U$1.A4
- removed net N$20: U$1.A5
- removed net N$22: U$1.RAW
- removed net N$6: LED1.A, R1.1
- new net BUZZER: C11.2, IC1A.QA, SG1.2
- new net ERROR_LED: IC1A.QH, R4.2
- new net LCD_BACKLIGHT: IC1A.QB, U1.K
- new net LCD_CLOCK: IC1A.SCK, U$1.*9
- new net LCD_DATA: IC1A.SER, U$1.A7
- new net LCD_ENABLE: IC1A.RCK, U$1.*10, U1.E
- new net N$7: IC1A.QE, U1.DB5
- new net SCL: CLOCK,TEMP,I2C.4, R1.2, U$1.A5
- new net SDA: CLOCK,TEMP,I2C.3, R5.2, U$1.A4
- new net TEMPERATURE_DS: CLOCK,TEMP,I2C.5
- new net TURN_WHEEL_A: SW1.A, U$1.2
- new net TURN_WHEEL_B: SW1.B, U$1.*3
- new net TURN_WHEEL_CLICK: SW1.SW+, U$1.4
- net +12V: now also R2.2; no longer LEDS3.1, LEDS4.1, R1.2
- net +5V/2: now also C10.+, C11.1, C3.1, CLOCK,TEMP,I2C.2, IC1A.SCL, IC1P.VCC, R1.1, R3.A, R5.1, SG1.1, U1.A, U1.VDD; no longer SWITCH.3
- net GND: now also C10.-, C3.2, CLOCK,TEMP,I2C.1, IC1A.G, IC1P.GND, POWER_SWITCH.P$1, R3.E, STATUS_LED.C, SW1.C, SW1.SW-, U1.R/W, U1.VSS; no longer LED1.C, LEDS3.3, LEDS4.3, SWITCH.1
- net LEDSTRIP1: now also U$1.*6
- net LEDSTRIP2: now also U$1.7
- net N$1: now also IC1A.QD, U1.DB4; no longer U$1.A6
- net N$10: now also U1.VO; no longer U$1.A3
- net N$11: now also R4.1, STATUS_LED.AR; no longer U$1.2
- net N$2: now also IC1A.QC, U1.RS; no longer U$1.A7
- net N$3: now also POWER_SWITCH.P$2, RN1D.1; no longer U$1.*10
- net N$5: now also R2.1, STATUS_LED.AG; no longer RN1D.1, SWITCH.2
- net N$8: now also IC1A.QF, U1.DB6; no longer U$1.A1
- net N$9: now also IC1A.QG, U1.DB7; no longer U$1.A2
- net POWER_SWITCH: now also U$1.*5
- net PROXIMITY: now also U$1.A3
- net PS_ON: now also U$1.A6
- net RF_DATA_IN: now also U$1.A1
- net RF_DATA_OUT: now also U$1.A2
Other:
- note added: "Contrast Tuning"
- note added: "Real Time Clock, Thermometer, I2C"
- note added: "Status Led"
- note removed: "Power Led"
- note removed: "Status Leds"
- moved on the sheet: C1, C2, R1, RN1D, SG1, SW1, U1

Commit message: Working on powernode layout.
Parts:
- removed C3: 100 nF, rcl:C-EUC0805
- removed RN1: 10k, resistor-dil:4R-N0603-ARC
- added C12: 100 nF, rcl:C-EUC0805
- added C13: 10 uF, rcl:C-EUC1206
- added R6: 4.7k, rcl:R-EU_R0805
- added R7: 1k, rcl:R-EU_R0805
- added R8: 2k, rcl:R-EU_R0805
- C10, C8, C9: device rcl:CPOL-EUE3.5-10 -> rcl:CPOL-EUE2.5-6
- C11: value 100 nF -> 100 uF; device rcl:C-EUC0805 -> rcl:CPOL-EUE2.5-6
Connections:
- removed net N$3: POWER_SWITCH.P$2, RN1D.1
- removed net N$4: RN1B.2, RN1C.2
- net +5V: now also BLUETOOTH.5, C11.+, C12.1, C13.1, ETHERNET.11, R3.A, R6.2, RF_RECEIVER.1, RF_TRANSMITTER.2, SG1.1, U1.A, U1.VDD
- net +5V/2: no longer BLUETOOTH.5, C11.1, C3.1, ETHERNET.11, R3.A, RF_RECEIVER.1, RF_TRANSMITTER.2, SG1.1, U1.A, U1.VDD
- net BLUETOOTH_RXD: now also R7.2; no longer RN1A.2
- net BUZZER: no longer C11.2
- net DATA_BUS: now also R6.1
- net GND: now also C11.-, C12.2, C13.2, R8.1; no longer C3.2, RN1C.1
- net N$21: now also R7.1, R8.2; no longer RN1A.1, RN1B.1
- net POWER_SWITCH: now also POWER_SWITCH.P$2; no longer RN1D.2
