File: lednode2.sch (EAGLE design)
At the start: 47 parts, among them Q1 AO3402, Q2 AO3402, Q3 AO3402, Q4 AO3402, Q5 AO3402, Q6 AO3402

Commit message: Working on new node version.
Parts:
- added C10: 100 nF, rcl:C-EUC0805
- added C11: 100 uF, rcl:CPOL-EUE2.5-6
- added C9: 10 uF, rcl:C-EUC1206
- added IC1: 74HCT595D, 74xx-eu:74HCT595D
- added SV1: (no value), con-lstb:MA04-2
Connections:
- new net +3V3: C10.1, C11.+, C9.1
- new net N$17: SV1.1
- new net N$18: SV1.3
- new net N$19: SV1.5
- new net N$20: SV1.7
- new net N$21: SV1.8
- new net N$22: SV1.6
- new net N$23: SV1.4
- new net N$24: SV1.2
- new net N$25: IC1A.RCK
- new net N$26: IC1A.SCK
- new net N$27: IC1A.SER
- net GND: now also C10.2, C11.-, C9.2
Other:
- note added: "(Temperature Sensor)"
- note added: "NRF24L01 Radio Module"
- note removed: "Temperature Sensor"
Changed lines of the file:
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@@
 <part name="SUPPLY64" library="supply2" deviceset="GND" device=""/>
 <part name="SUPPLY65" library="supply2" deviceset="+12V" device=""/>
+<part name="SV1" library="con-lstb" deviceset="MA04-2" device=""/>
+<part name="IC1" library="74xx-eu" deviceset="74*595" device="D" technology="HCT"/>
+<part name="SUPPLY40" library="supply2" deviceset="GND" device=""/>
+<part name="C9" library="rcl" deviceset="C-EU" device="C1206" value="10 uF"/>
+<part name="C10" library="rcl" deviceset="C-EU" device="C0805" value="100 nF"/>
+<part name="+3V1" library="supply1" deviceset="+3V3" device=""/>
+<part name="C11" library="rcl" deviceset="CPOL-EU" device="E2.5-6" value="100 uF"/>
 </parts>
 <sheets>
@@
 <text x="-111.76" y="-22.86" size="2.54" layer="91">Extra Inputs</text>
 <text x="-111.76" y="68.58" size="2.54" layer="91">Vibration Sensor</text>
-<text x="-170.18" y="20.32" size="2.54" layer="91">Temperature Sensor</text>
+<text x="-170.18" y="20.32" size="2.54" layer="91">(Temperature Sensor)</text>
 <text x="-15.24" y="60.96" size="2.54" layer="91">Power Connector</text>
 <text x="132.08" y="83.82" size="2.54" layer="91">Spotlight Drivers</text>
 <text x="-111.76" y="15.24" size="2.54" layer="91">Sound Sensor</text>
 <text x="-63.5" y="30.48" size="2.1844" layer="91">Breakouts for unused pins</text>
+<text x="-66.04" y="91.44" size="2.54" layer="91">NRF24L01 Radio Module</text>
 </plain>
 <instances>
@@
 <instance part="SUPPLY64" gate="GND" x="5.08" y="48.26" rot="R90"/>
 <instance part="SUPPLY65" gate="+12V" x="5.08" y="50.8" rot="R270"/>
+<instance part="SV1" gate="G$1" x="-48.26" y="78.74"/>
+<instance part="IC1" gate="A" x="93.98" y="86.36"/>
+<instance part="SUPPLY40" gate="GND" x="33.02" y="-93.98"/>
+<instance part="C9" gate="G$1" x="25.4" y="-86.36"/>
+<instance part="C10" gate="G$1" x="40.64" y="-86.36"/>
+<instance part="+3V1" gate="G$1" x="40.64" y="-76.2"/>
+<instance part="C11" gate="G$1" x="53.34" y="-86.36"/>
 </instances>
 <busses>
@@
 <pinref part="SUPPLY64" gate="GND" pin="GND"/>
 </segment>
+<segment>
+<pinref part="C9" gate="G$1" pin="2"/>
+<pinref part="SUPPLY40" gate="GND" pin="GND"/>
+<wire x1="25.4" y1="-91.44" x2="33.02" y2="-91.44" width="0.1524" layer="91"/>
+<pinref part="C10" gate="G$1" pin="2"/>
+<wire x1="33.02" y1="-91.44" x2="40.64" y2="-91.44" width="0.1524" layer="91"/>
+<junction x="33.02" y="-91.44"/>
+<pinref part="C11" gate="G$1" pin="-"/>
+<wire x1="53.34" y1="-91.44" x2="40.64" y2="-91.44" width="0.1524" layer="91"/>
+<junction x="40.64" y="-91.44"/>
+</segment>
 </net>
 <net name="+5V" class="0">
@@
 </segment>
 </net>
+<net name="N$17" class="0">
+<segment>
+<pinref part="SV1" gate="G$1" pin="1"/>
+<wire x1="-40.64" y1="73.66" x2="-17.78" y2="73.66" width="0.1524" layer="91"/>
+<label x="-38.1" y="73.66" size="1.778" layer="95"/>
+</segment>
+</net>
+<net name="N$18" class="0">
+<segment>
+<pinref part="SV1" gate="G$1" pin="3"/>
+<wire x1="-40.64" y1="76.2" x2="-17.78" y2="76.2" width="0.1524" layer="91"/>
+<label x="-38.1" y="76.2" size="1.778" layer="95"/>
+</segment>
+</net>
+<net name="N$19" class="0">
+<segment>
+<pinref part="SV1" gate="G$1" pin="5"/>
+<wire x1="-40.64" y1="78.74" x2="-17.78" y2="78.74" width="0.1524" layer="91"/>
+<label x="-38.1" y="78.74" size="1.778" layer="95"/>
+</segment>
+</net>
+<net name="N$20" class="0">
+<segment>
+<pinref part="SV1" gate="G$1" pin="7"/>
+<wire x1="-40.64" y1="81.28" x2="-17.78" y2="81.28" width="0.1524" layer="91"/>
+<label x="-38.1" y="81.28" size="1.778" layer="95"/>
+</segment>
+</net>
+<net name="N$21" class="0">
+<segment>
+<pinref part="SV1" gate="G$1" pin="8"/>
+<wire x1="-55.88" y1="81.28" x2="-81.28" y2="81.28" width="0.1524" layer="91"/>
+<label x="-81.28" y="81.28" size="1.778" layer="95"/>
+</segment>
+</net>
+<net name="N$22" class="0">
+<segment>
+<pinref part="SV1" gate="G$1" pin="6"/>
+<wire x1="-55.88" y1="78.74" x2="-81.28" y2="78.74" width="0.1524" layer="91"/>
+<label x="-81.28" y="78.74" size="1.778" layer="95"/>
+</segment>
+</net>
+<net name="N$23" class="0">
+<segment>
+<pinref part="SV1" gate="G$1" pin="4"/>
+<wire x1="-55.88" y1="76.2" x2="-81.28" y2="76.2" width="0.1524" layer="91"/>
+<label x="-81.28" y="76.2" size="1.778" layer="95"/>
+</segment>
+</net>
+<net name="N$24" class="0">
+<segment>
+<pinref part="SV1" gate="G$1" pin="2"/>
+<wire x1="-55.88" y1="73.66" x2="-81.28" y2="73.66" width="0.1524" layer="91"/>
+<label x="-81.28" y="73.66" size="1.778" layer="95"/>
+</segment>
+</net>
+<net name="N$25" class="0">
+<segment>
+<pinref part="IC1" gate="A" pin="RCK"/>
+<wire x1="81.28" y1="83.82" x2="55.88" y2="83.82" width="0.1524" layer="91"/>
+</segment>
+</net>
+<net name="N$26" class="0">
+<segment>
+<pinref part="IC1" gate="A" pin="SCK"/>
+<wire x1="81.28" y1="91.44" x2="55.88" y2="91.44" width="0.1524" layer="91"/>
+</segment>
+</net>
+<net name="N$27" class="0">
+<segment>
+<pinref part="IC1" gate="A" pin="SER"/>
+<wire x1="81.28" y1="96.52" x2="55.88" y2="96.52" width="0.1524" layer="91"/>
+</segment>
+</net>
+<net name="+3V3" class="0">
+<segment>
+<pinref part="C9" gate="G$1" pin="1"/>
+<pinref part="C10" gate="G$1" pin="1"/>
+<wire x1="25.4" y1="-83.82" x2="40.64" y2="-83.82" width="0.1524" layer="91"/>
+<pinref part="+3V1" gate="G$1" pin="+3V3"/>
+<wire x1="40.64" y1="-78.74" x2="40.64" y2="-83.82" width="0.1524" layer="91"/>
+<junction x="40.64" y="-83.82"/>
+<pinref part="C11" gate="G$1" pin="+"/>
+<wire x1="53.34" y1="-83.82" x2="40.64" y2="-83.82" width="0.1524" layer="91"/>
+<junction x="40.64" y="-83.82"/>
+</segment>
+</net>

Commit message: Working on lednode v2.0
Parts:
- removed IC1: 74HCT595D, 74xx-eu:74HCT595D
- removed LEDS6: (no value), SparkFun-Connectors:M03LONGPADS
- removed Q6: AO3402, adafruit:MOSFET-NWAVE
- removed R1, R2, R3: 10k, rcl:R-EU_R0805
- removed SENSOR1, SENSOR2: (no value), SparkFun-Connectors:M03PTH
- removed SHAKE: SW-18010P, sensor-comus-group:CM4400
- removed SPOT6: M025MM, SparkFun-Connectors:M025MM
- removed SV1: (no value), con-lstb:MA04-2
- removed THERM: 10k, discrete-fixed-thermistor-silk:THERMISTOR_R-7,5
- added 3.3V_REGULATOR: AMS1117-3.3, burr-brown:REG1117
- added C12: 22uF, Tantalum, rcl:CPOL-EUSMCA
- added C13: (22uF, Tantalum), rcl:CPOL-EUSMCA
- added C14, C15: 100 uF, rcl:CPOL-EUE2.5-6
- added IO1, IO2: (no value), SparkFun-Connectors:M03PTH
- added L1: WS2812B, adafruit:WS2812B
- added POWERLED: (no value), led:LEDSMT1206
- added RADIO: NRF24L01, con-lstb:MA04-2
- C9: value 10 uF -> 100 uF; device rcl:C-EUC1206 -> rcl:CPOL-EUE2.5-6
Connections:
- net EXTRA_SENSOR1 renamed EXTRA_IO1
- net EXTRA_SENSOR2 renamed EXTRA_IO2
- removed net DATA_BUS: U$1.A0
- removed net LEDSTRIP6: LEDS6.2, U$1.A2
- removed net N$12: Q6.G, RN3D.2
- removed net N$17: SV1.1
- removed net N$18: SV1.3
- removed net N$19: SV1.5
- removed net N$20: SV1.7
- removed net N$21: SV1.8
- removed net N$22: SV1.6
- removed net N$23: SV1.4
- removed net N$24: SV1.2
- removed net N$25: IC1A.RCK
- removed net N$26: IC1A.SCK
- removed net N$27: IC1A.SER
- removed net SHAKE: R1.2, SHAKE.1, U$1.12
- removed net SPOTLIGHT6: RN3D.1, RN4D.2, U$1.*11
- removed net TEMPERATURE: R2.2, THERM.2, U$1.A6
- new net RADIO_CE: RADIO.3, U$1.A1
- new net RADIO_CSN: RADIO.4, U$1.A0
- new net RADIO_IRQ: RADIO.8
- new net RADIO_MISO: RADIO.7, U$1.12
- new net RADIO_MOSI: RADIO.6, U$1.*11
- new net RADIO_SCK: RADIO.5, U$1.13
- new net STATUS_AND_LEDSTRIP5: L1.DIN, U$1.A3
- net +12V: now also 3.3V_REGULATOR.VIN, C13.+, C14.+, C9.+; no longer LEDS6.1, SPOT6.1
- net +3V3: now also 3.3V_REGULATOR.VOUT, C12.+, POWERLED.A, RADIO.2; no longer C9.1
- net +5V: now also C15.+, IO1.3, IO2.3, L1.VDD; no longer SENSOR1.3, SENSOR2.3, SHAKE.2, THERM.1
- net GND: now also 3.3V_REGULATOR.GND, C12.-, C13.-, C14.-, C15.-, C9.-, IO1.1, IO2.1, L1.GND, RADIO.1, RN3D.1; no longer C9.2, LEDS6.3, Q6.S, R1.1, R2.1, R3.1, SENSOR1.1, SENSOR2.1
- net LEDSTRIP1: now also U$1.2; no longer U$1.4
- net LEDSTRIP2: now also U$1.4; no longer U$1.2
- net LEDSTRIP5: now also L1.DOUT; no longer U$1.A1
- net LIGHTLEVEL: now also RN4D.2; no longer R3.2
- net N$11: now also POWERLED.C, RN3D.2; no longer Q6.D, SPOT6.2
- net N$13: now also IO2.2; no longer SENSOR2.2
- net PROXIMITY: now also U$1.A6; no longer U$1.13
- net SENSOR1: now also IO1.2; no longer SENSOR1.2
- net SOUND_ANALOG: now also U$1.A2; no longer U$1.A3
Other:
- note added: "3.3V Regulator"
- note added: "Extra Inputs / Outputs"
- note added: "NOTE: The regulator needs at least a 10mA load to work, and the radio may draw less than that, so we add the power led on the 3.3V rail."
- note added: "Status LED"
- note added: "TODO: Check if the yellow-green smd leds work with 3.3V and a 220 Ohm resistor."
- note removed: "(Temperature Sensor)"
- note removed: "Extra Inputs"
- note removed: "Vibration Sensor"
- moved on the sheet: C10, C11, C7, C8, LEDS1, LEDS2, LEDS3, LEDS4, LEDS5, PHOTOCELL, PIR, POWER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

Commit message: tuning.
Connections:
- new net N$12: RN4C.1, RN4D.1
- new net N$17: RN4B.2, RN4C.2
- net GND: no longer RN4C.1, RN4D.1
- net N$13: no longer RN2D.2
- net SENSOR1: no longer RN4A.2
- net SPOTLIGHT4: now also RN2D.2; no longer RN4B.2
- net SPOTLIGHT5: now also RN4A.2; no longer RN4C.2
Other:
- moved on the sheet: IO1, IO2, PHOTOCELL, RN1D, RN2D, RN3A, RN4A, RN4B, RN4C, RN4D
